Commit message: Update Gazebo launch configuration and add new controllers for impedance handling

File: lbr_description/gazebo/lbr_gazebo.xacro (robot description, xacro)
@@ -6,5 +6,5 @@
             <plugin name="ign_ros2_control::IgnitionROS2ControlPlugin"
                 filename="ign_ros2_control-system">
-                <parameters>$(find lbr_description)/ros2_control/lbr_controllers.yaml</parameters>
+                <parameters>$(find lbr_description)/ros2_control/lbr_gazebo_controllers.yaml</parameters>
                 <ros>
                     <namespace>/${robot_name}</namespace>
@@ -13,4 +13,8 @@
                     <remapping>cartesian_impedance_controller/target_frame:=target_frame</remapping>
                     <remapping>cartesian_impedance_controller/target_wrench:=target_wrench</remapping>
+                    <remapping>cbf_cartesian_impedance_controller/target_frame:=target_frame</remapping>
+                    <remapping>cbf_cartesian_impedance_controller/target_wrench:=target_wrench</remapping>
+                    <remapping>hocbf_cartesian_impedance_controller/target_frame:=target_frame</remapping>
+                    <remapping>hocbf_cartesian_impedance_controller/target_wrench:=target_wrench</remapping>
                     <remapping>joint_impedance_controller/target_frame:=target_frame</remapping>
                     <remapping>joint_impedance_controller/target_wrench:=target_wrench</remapping>

File: lbr_description/urdf/iiwa14/iiwa14_description.xacro (robot description, xacro)
@@ -253,5 +253,5 @@
                 <origin rpy="0 0 0" xyz="-0.0029 8.1e-04 0.1998" />
                 <mass value="3.5296" />
-                <inertia ixx="0.0081" ixy="-9.1e-06" ixz="-9.9e-06" iyy="1.0e-04" iyz="-9.9e-06"
+                <inertia ixx="0.0081" ixy="-9.1e-06" ixz="-9.9e-06" iyy="1.2e-04" iyz="-9.9e-06"
                     izz="0.0080" />
                 <!-- iyy is 1.0e.05 in the paper but it seems to cause invalid inertia error -->

Commit message: Add kuka_cartesian_impedance_controller and update configurations for improved control

File: lbr_description/gazebo/lbr_gazebo.xacro (robot description, xacro)
@@ -17,4 +17,6 @@
                     <remapping>hocbf_cartesian_impedance_controller/target_frame:=target_frame</remapping>
                     <remapping>hocbf_cartesian_impedance_controller/target_wrench:=target_wrench</remapping>
+                    <remapping>kuka_cartesian_impedance_controller/target_frame:=target_frame</remapping>
+                    <remapping>kuka_cartesian_impedance_controller/target_wrench:=target_wrench</remapping>
                     <remapping>joint_impedance_controller/target_frame:=target_frame</remapping>
                     <remapping>joint_impedance_controller/target_wrench:=target_wrench</remapping>

File: lbr_description/urdf/ultrasound_probe/bota_camera_ultrasound.xacro (robot description, xacro)
@@ -130,5 +130,5 @@
     <parent link="$(arg robot_name)_link_ee" />
     <child link="probe" />
-    <origin xyz="0.0 0.0 0.16" rpy="0.0 0.0 -${pi/4}" />
+    <origin xyz="0.0 0.0 0.17" rpy="0.0 0.0 -${pi/4}" />
   </joint>
 </robot>
