Commit message: simplified clarius mesh and fixed frames

File: lbr_description/urdf/ultrasound_probe/ultrasound_clarius.xacro (robot description, xacro)
@@ -3,5 +3,5 @@
 <robot name="iiwa14" xmlns:xacro="http://www.ros.org/wiki/xacro">
   <material name="transparent">
-    <color rgba="1 0 0 1.0" />
+    <color rgba="0.2 0.2 0.2 0.1" />
   </material>
   <!-- include the lbr iiwa macro -->
@@ -34,7 +34,7 @@
     <parent link="$(arg robot_name)_link_ee" />
     <child link="clarius_holder" />
-    <origin xyz="0.0 0.0 0.0" rpy="0.0 0.0 0.0" />
+    <origin xyz="0.0 0.0 0.0" rpy="0.0 0.0 ${pi}" />
   </joint>
-  <!-- US probe model -->
+  <!-- US holder model -->
   <link
     name="clarius_holder">
@@ -45,10 +45,25 @@
           scale="0.001 0.001 0.001" />
       </geometry>
-      <material
-        name="">
-        <color
-          rgba="0.2 0.2 0.2 1" />
-      </material>
+      <material name="transparent"/>
     </visual>
+  </link>
+  <!-- US probe model -->
+  <joint name="clarius_joint" type="fixed">
+    <parent link="clarius_holder" />
+    <child link="clarius_probe" />
+    <origin xyz="0.0 0.0 0.0" rpy="0.0 0.0 0.0" />
+  </joint>
+  <link
+  name="clarius_probe">
+  <visual>
+    <origin xyz="0 0 0" rpy="0 0 0" />
+    <geometry>
+      <mesh filename="package://lbr_description/meshes/ultrasound_probe/clarius.stl"
+        scale="0.001 0.001 0.001" />
+    </geometry>
+    <material name="grey">
+      <color rgba="1.0 1.0 1.0 1.0" />
+    </material>
+  </visual>
   </link>
   <!-- <link
@@ -66,5 +81,5 @@
     <parent link="$(arg robot_name)_link_ee" />
     <child link="probe" />
-    <origin xyz="0.0 0.0 0.175" rpy="0.0 0.0 -${pi/2}" />
+    <origin xyz="0.0 0.013 0.145" rpy="0.0 -0.610865 -${pi/2}" />
   </joint>
 </robot>

Commit message: modified clarius probe pose

File: lbr_description/urdf/ultrasound_probe/ultrasound_clarius.xacro (robot description, xacro)
@@ -3,5 +3,5 @@
 <robot name="iiwa14" xmlns:xacro="http://www.ros.org/wiki/xacro">
   <material name="transparent">
-    <color rgba="0.2 0.2 0.2 0.1" />
+    <color rgba="0.2 0.2 0.2 1.0" />
   </material>
   <!-- include the lbr iiwa macro -->
@@ -34,5 +34,5 @@
     <parent link="$(arg robot_name)_link_ee" />
     <child link="clarius_holder" />
-    <origin xyz="0.0 0.0 0.0" rpy="0.0 0.0 ${pi}" />
+    <origin xyz="0.0 0.0 0.0" rpy="0.0 0.0 ${-pi/2}" />
   </joint>
   <!-- US holder model -->
@@ -45,5 +45,5 @@
           scale="0.001 0.001 0.001" />
       </geometry>
-      <material name="transparent"/>
+      <material name="transparent" />
     </visual>
   </link>
@@ -51,19 +51,26 @@
   <joint name="clarius_joint" type="fixed">
     <parent link="clarius_holder" />
-    <child link="clarius_probe" />
-    <origin xyz="0.0 0.0 0.0" rpy="0.0 0.0 0.0" />
+    <child link="probe" />
+    <origin xyz="0.0 -0.0135 0.145" rpy="0.610865 0.0 0.0" />
+  </joint>
+  <joint name="clarius_joint_visual" type="fixed">
+    <parent link="clarius_holder" />
+    <child link="probe_visual" />
+    <origin xyz="0.0 0.00 0.0" rpy="0 0.0 0.0" />
   </joint>
   <link
-  name="clarius_probe">
-  <visual>
-    <origin xyz="0 0 0" rpy="0 0 0" />
-    <geometry>
-      <mesh filename="package://lbr_description/meshes/ultrasound_probe/clarius.stl"
-        scale="0.001 0.001 0.001" />
-    </geometry>
-    <material name="grey">
-      <color rgba="1.0 1.0 1.0 1.0" />
-    </material>
-  </visual>
+    name="probe_visual">
+    <visual>
+      <geometry>
+        <mesh filename="package://lbr_description/meshes/ultrasound_probe/clarius.stl"
+          scale="0.001 0.001 0.001" />
+      </geometry>
+      <material name="grey">
+        <color rgba="1.0 1.0 1.0 1.0" />
+      </material>
+    </visual>
+  </link>
+  <link
+    name="probe">
   </link>
   <!-- <link
@@ -75,11 +82,11 @@
     <origin xyz="0.0 0.0 0.14" rpy="0.0 0.0 0.0" />
   </joint> -->
-  <link
+  <!-- <link
     name="probe">
   </link>
   <joint name="probe_transl_joint" type="fixed">
-    <parent link="$(arg robot_name)_link_ee" />
+    <parent link="clarius_probe" />
     <child link="probe" />
-    <origin xyz="0.0 0.013 0.145" rpy="0.0 -0.610865 -${pi/2}" />
-  </joint>
+    <origin xyz="0.0 0.0 0.0" rpy="0 0.0 0.0" />
+  </joint> -->
 </robot>
