Commit message: working branch

File: lbr_description/urdf/iiwa14/iiwa14_description.xacro (robot description, xacro)
@@ -271,4 +271,11 @@
         <link name="link_ee">
         </link>
+        <joint name="joint_tool" type="fixed">
+            <parent link="link_ee" />
+            <child link="link_tool" />
+            <origin xyz="0 0 0.01" rpy="0 0 0" />
+        </joint>
+        <link name="link_tool">
+        </link>
     </xacro:macro>
 </robot>

Commit message: minor

File: lbr_description/urdf/iiwa14/iiwa14_description.xacro (robot description, xacro)
@@ -1,3 +1,4 @@
 <?xml version="1.0"?>
+<!-- Using masses and inertia matrices from this paper https://ieeexplore.ieee.org/document/9112185 -->
 <robot xmlns:xacro="http://www.ros.org/wiki/xacro">
     <!-- robot as extracted via https://github.com/syuntoku14/fusion2urdf -->
@@ -56,8 +57,8 @@
         <link name="${robot_name}_link_1">
             <inertial>
-                <origin rpy="0 0 0" xyz="0.0 -0.033795 0.132404" />
-                <mass value="5.289529" />
-                <inertia ixx="0.042462" ixy="0.0" ixz="0.0" iyy="0.042838" iyz="0.006341"
-                    izz="0.01587" />
+                <origin rpy="0 0 0" xyz="-0.018 0.0455 -0.1050" />
+                <mass value="1.0" />
+                <inertia ixx="0.5468" ixy="-0.0082" ixz="0.0116" iyy="0.6997" iyz="-0.0136"
+                    izz="0.1625" />
             </inertial>
             <visual>
@@ -88,8 +89,8 @@
         <link name="${robot_name}_link_2">
             <inertial>
-                <origin rpy="0 0 0" xyz="0.000136 0.047548 0.076322" />
-                <mass value="5.688888" />
-                <inertia ixx="0.055182" ixy="-3.3e-05" ixz="5.6e-05" iyy="0.053983" iyz="0.010034"
-                    izz="0.016523" />
+                <origin rpy="0 0 0" xyz="0.0219 0.1218 0.0500" />
+                <mass value="5.5609" />
+                <inertia ixx="0.0022" ixy="7.3e-05" ixz="-7.3e-05" iyy="7.3e-04" iyz="-7.3e-05"
+                    izz="0.0029" />
             </inertial>
             <visual>
@@ -120,8 +121,9 @@
         <link name="${robot_name}_link_3">
             <inertial>
-                <origin rpy="0 0 0" xyz="0.0 0.034913 0.123108" />
-                <mass value="3.461245" />
-                <inertia ixx="0.02172" ixy="0.0" ixz="0.0" iyy="0.02073" iyz="-0.003845"
-                    izz="0.007701" />
+                <origin rpy="0 0 0" xyz="-0.0216 0.0500 -0.3000" />
+                <mass value="5.9199" />
+                <inertia ixx="3.0e-04" ixy="-5.4e-06" ixz="-1.0e-05" iyy="4.0e-04" iyz="-9.8e-06"
+                    izz="1.02e-04" />
+                <!-- izz is 1.0e.04 in the paper but it seems to cause invalid inertia error -->
             </inertial>
             <visual>
@@ -152,8 +154,9 @@
         <link name="${robot_name}_link_4">
             <inertial>
-                <origin rpy="0 0 0" xyz="0.0 -0.039793 0.086944" />
-                <mass value="4.122995" />
-                <inertia ixx="0.03241" ixy="0.0" ixz="0.0" iyy="0.030758" iyz="-0.006022"
-                    izz="0.009883" />
+                <origin rpy="0 0 0" xyz="0.0161 -0.2004 -0.0425" />
+                <mass value="6.0000" />
+                <inertia ixx="3.0e-04" ixy="-9.9e-06" ixz="9.9e-06" iyy="1.03e-04" iyz="-1.0e-05"
+                    izz="4.0e-04" />
+                <!-- iyy is 1.0e.05 in the paper but it seems to cause invalid inertia error -->
             </inertial>
             <visual>
@@ -184,8 +187,8 @@
         <link name="${robot_name}_link_5">
             <inertial>
-                <origin rpy="0 0 0" xyz="0.0 -0.029824 0.076267" />
-                <mass value="1.563756" />
-                <inertia ixx="0.008677" ixy="0.0" ixz="0.0" iyy="0.007297" iyz="0.002869"
-                    izz="0.003935" />
+                <origin rpy="0 0 0" xyz="0.00056 0.0131 -0.2390" />
+                <mass value="2.9896" />
+                <inertia ixx="3.0e-04" ixy="1.0e-05" ixz="-9.8e-06" iyy="3.0e-04" iyz="9.8e-06"
+                    izz="1.0e-04" />
             </inertial>
             <visual>
@@ -216,8 +219,8 @@
         <link name="${robot_name}_link_6">
             <inertial>
-                <origin rpy="0 0 0" xyz="0.0 0.07102 0.00495" />
-                <mass value="2.457878" />
-                <inertia ixx="0.007227" ixy="0.0" ixz="0.0" iyy="0.006958" iyz="0.000318"
-                    izz="0.004734" />
+                <origin rpy="0 0 0" xyz="0.0074 0.1500 -0.0232" />
+                <mass value="1.0000" />
+                <inertia ixx="1.0e-04" ixy="-9.9e-06" ixz="-1.0e-05" iyy="1.0e-04" iyz="9.9e-06"
+                    izz="1.0e-04" />
             </inertial>
             <visual>
@@ -248,7 +251,9 @@
         <link name="${robot_name}_link_7">
             <inertial>
-                <origin rpy="0 0 0" xyz="3.0000e-06 -2.0000e-06 1.3782e-02" />
-                <mass value="0.265331" />
-                <inertia ixx="0.000175" ixy="0.0" ixz="0.0" iyy="0.000175" iyz="0.0" izz="0.000306" />
+                <origin rpy="0 0 0" xyz="-0.0029 8.1e-04 0.1998" />
+                <mass value="3.5296" />
+                <inertia ixx="0.0081" ixy="-9.1e-06" ixz="-9.9e-06" iyy="1.0e-04" iyz="-9.9e-06"
+                    izz="0.0080" />
+                <!-- iyy is 1.0e.05 in the paper but it seems to cause invalid inertia error -->
             </inertial>
             <visual>

Commit message: updated probe mesh and rate

File: lbr_description/urdf/iiwa14/iiwa14_description.xacro (robot description, xacro)
@@ -35,4 +35,5 @@
                     <mesh filename="package://lbr_description/meshes/iiwa14/visual/link_0.dae" />
                 </geometry>
+                <material name="transparent"/>
             </visual>
             <collision>
@@ -67,4 +68,5 @@
                     <mesh filename="package://lbr_description/meshes/iiwa14/visual/link_1.dae" />
                 </geometry>
+                <material name="transparent"/>
             </visual>
             <collision>
@@ -99,4 +101,5 @@
                     <mesh filename="package://lbr_description/meshes/iiwa14/visual/link_2.dae" />
                 </geometry>
+                <material name="transparent"/>
             </visual>
             <collision>
@@ -132,4 +135,5 @@
                     <mesh filename="package://lbr_description/meshes/iiwa14/visual/link_3.dae" />
                 </geometry>
+                <material name="transparent"/>
             </visual>
             <collision>
@@ -165,4 +169,5 @@
                     <mesh filename="package://lbr_description/meshes/iiwa14/visual/link_4.dae" />
                 </geometry>
+                <material name="transparent"/>
             </visual>
             <collision>
@@ -197,4 +202,5 @@
                     <mesh filename="package://lbr_description/meshes/iiwa14/visual/link_5.dae" />
                 </geometry>
+                <material name="transparent"/>
             </visual>
             <collision>
@@ -229,4 +235,5 @@
                     <mesh filename="package://lbr_description/meshes/iiwa14/visual/link_6.dae" />
                 </geometry>
+                <material name="transparent"/>
             </visual>
             <collision>
@@ -262,4 +269,5 @@
                     <mesh filename="package://lbr_description/meshes/iiwa14/visual/link_7.dae" />
                 </geometry>
+                <material name="transparent"/>
             </visual>
             <collision>

File: lbr_description/urdf/ultrasound_probe/ultrasound_atl.xacro (robot description, xacro)
@@ -2,30 +2,33 @@
 <!-- top level -->
 <robot name="iiwa14" xmlns:xacro="http://www.ros.org/wiki/xacro">
-    <!-- include the lbr iiwa macro -->
-    <xacro:include filename="$(find lbr_description)/urdf/iiwa14/iiwa14_description.xacro" />
-    <xacro:arg name="robot_name" default="lbr" />
-    <xacro:arg name="mode" default="true" />
-    <!-- <xacro:arg name="use_ft_sensor" default="true" /> -->
-    <xacro:arg
-        name="system_config_path"
-        default="$(find lbr_description)/ros2_control/lbr_system_config.yaml" />
-    <!-- KDL requires a link without inertia -->
-    <link name="$(arg robot_name)_floating_link" />
-    <link name="world" />
-    <joint name="$world_to_base" type="fixed">
-        <parent link="world" />
-        <child link="$(arg robot_name)_floating_link" />
-    </joint>
-    <!--joint
+  <material name="transparent">
+    <color rgba="1 0 0 1.0" />
+  </material>
+  <!-- include the lbr iiwa macro -->
+  <xacro:include filename="$(find lbr_description)/urdf/iiwa14/iiwa14_description.xacro" />
+  <xacro:arg name="robot_name" default="lbr" />
+  <xacro:arg name="mode" default="true" />
+  <!-- <xacro:arg name="use_ft_sensor" default="true" /> -->
+  <xacro:arg
+    name="system_config_path"
+    default="$(find lbr_description)/ros2_control/lbr_system_config.yaml" />
+  <!-- KDL requires a link without inertia -->
+  <link name="$(arg robot_name)_floating_link" />
+  <link name="world" />
+  <joint name="$world_to_base" type="fixed">
+    <parent link="world" />
+    <child link="$(arg robot_name)_floating_link" />
+  </joint>
+  <!--joint
         between <robot_name>_floating_link and robot_name_link_0-->
-    <joint name="$(arg robot_name)_floating_joint" type="fixed">
-        <parent link="$(arg robot_name)_floating_link" />
-        <child link="$(arg robot_name)_link_0" />
-    </joint>
-    <!-- iiwa -->
-    <xacro:iiwa14
-        robot_name="$(arg robot_name)"
-        mode="$(arg mode)"
-        system_config_path="$(arg system_config_path)" />
+  <joint name="$(arg robot_name)_floating_joint" type="fixed">
+    <parent link="$(arg robot_name)_floating_link" />
+    <child link="$(arg robot_name)_link_0" />
+  </joint>
+  <!-- iiwa -->
+  <xacro:iiwa14
+    robot_name="$(arg robot_name)"
+    mode="$(arg mode)"
+    system_config_path="$(arg system_config_path)" />
   <!-- force sensor urdf -->
   <!-- <xacro:include filename="$(find rokubimini_description)/urdf/BFT_SENS_ECAT_M8.urdf.xacro" /> -->
@@ -49,6 +52,7 @@
         name="">
         <color
-          rgba="0.6902 0.61176 0.52941 1" />
+          rgba="0.6902 0.61176 0.52941 0" />
       </material>
+      <material name="transparent" />
     </visual>
   </link>
@@ -56,5 +60,5 @@
     <parent link="$(arg robot_name)_link_ee" />
     <child link="camera_support" />
-    <origin xyz="0.00 0.00 0.005" rpy="-${pi/2} ${pi} ${1*pi/4}" />
+    <origin xyz="0.00 0.00 0.005" rpy="-${pi/2} ${pi} ${2*pi/4}" />
   </joint>
   <!-- ZED -->
@@ -68,17 +72,18 @@
   <xacro:arg name="camera_model" default="zed2" />
   <xacro:arg name="custom_baseline" default="0.0" />
-  <joint name="camera_support_joint2" type="fixed">
-    <parent link="camera_support" />
-    <child link="zed2_camera_link" />
-    <origin xyz="-0.081653 0.018797 0.0" rpy="-${pi/2} 0.0 ${pi/2}" />
-  </joint>
+  <!-- <origin xyz="-0.081653 0.018797 0.0" rpy="-${pi/2} 0.0 ${pi/2}" /> -->
   <!-- <joint name="camera_support_joint2" type="fixed">
     <parent link="camera_support" />
     <child link="zed2_camera_link" />
-    <origin xyz="-0.081653 0.045 0.0" rpy="-${pi/2} 0.0 ${pi/2}" />
+    <origin xyz="-0.081653 0.040 0.0" rpy="-${pi/2} 0.0 ${pi/2}" />
+  </joint> -->
+  <!-- <joint name="camera_support_joint2" type="fixed">
+    <parent link="camera_support" />
+    <child link="zed2_camera_link" />
+    <origin xyz="-0.081653 0.016 0.0" rpy="-${pi/2} 0.0 ${pi/2}" />
   </joint> -->
   <!-- If GNSS fusion is enabled the position of the antenna with respect to the camera mount point
   is required -->
-  <xacro:arg name="enable_gnss" default="false" />
+  <!-- <xacro:arg name="enable_gnss" default="false" />
   <xacro:arg name="gnss_x" default="0.0" />
   <xacro:arg name="gnss_y" default="0.0" />
@@ -88,31 +93,31 @@
     custom_baseline="$(arg custom_baseline)" enable_gnss="$(arg enable_gnss)">
     <origin xyz="$(arg gnss_x) $(arg gnss_y) $(arg gnss_z)" rpy="0 0 0" />
-  </xacro:zed_camera>
+  </xacro:zed_camera> -->
   <joint name="camera_to_probe" type="fixed">
     <parent link="camera_support" />
     <child link="probe_mounting" />
-    <origin xyz="0 0 0" rpy="-${pi/2} ${-pi/4} 0.0" />
+    <origin xyz="0 0 0" rpy="-${pi/2} ${0.0} 0.0" />
   </joint>
   <!-- US probe model -->
   <link
-  name="probe_mounting">
-  <inertial>
-    <origin rpy="0 0 0" xyz="0.0204 0.0212 0.0492" />
-    <mass value="0.5" />
-    <inertia ixx="0.044604" ixy="0.0" ixz="-0.000788" iyy="0.045465" iyz="0.0"
+    name="probe_mounting">
+    <inertial>
+      <origin rpy="0 0 0" xyz="0.0204 0.0212 0.0492" />
+      <mass value="0.5" />
+      <inertia ixx="0.044604" ixy="0.0" ixz="-0.000788" iyy="0.045465" iyz="0.0"
         izz="0.061904" />
-</inertial>
-  <visual>
-    <origin xyz="0 0 0" rpy="0 0 0" />
-    <geometry>
-      <mesh filename="package://lbr_description/meshes/ultrasound_probe/probe.stl"
-        scale="0.001 0.001 0.001" />
-    </geometry>
-    <material
-      name="">
-      <color
-        rgba="0.2 0.2 0.2 1" />
-    </material>
-  </visual>
+    </inertial>
+    <visual>
+      <origin xyz="0 0 0" rpy="0 0 0" />
+      <geometry>
+        <mesh filename="package://lbr_description/meshes/ultrasound_probe/probe.stl"
+          scale="0.001 0.001 0.001" />
+      </geometry>
+      <material
+        name="">
+        <color
+          rgba="0.2 0.2 0.2 1" />
+      </material>
+    </visual>
   </link>
   <!-- <link
@@ -125,10 +130,10 @@
   </joint> -->
   <link
-  name="probe">
+    name="probe">
   </link>
   <joint name="probe_transl_joint" type="fixed">
     <parent link="$(arg robot_name)_link_ee" />
     <child link="probe" />
-    <origin xyz="0.0 0.0 0.175" rpy="0.0 0.0 -${pi/4}" />
+    <origin xyz="0.0 0.0 0.175" rpy="0.0 0.0 -${pi/2}" />
   </joint>
 </robot>
